Commit message: put correct

File: catkin_yuhaow7/src/drivers/diff_wheeled_robot_gazebo/urdf/diff_wheeled_robot.xacro (robot description, xacro)
@@ -9,6 +9,6 @@
     <color rgba="0.8 0.0 0.0 1.0"/>
   </material>
-  <material name="White">
-    <color rgba="1.0 1.0 1.0 1.0"/>
+  <material name="Purple">
+    <color rgba="0.5 0.0 1.0 1.0"/>
   </material>
   <material name="Blue">
@@ -90,5 +90,5 @@
           <cylinder length="${base_height}" radius="${base_radius}" />
       </geometry>
-      <material name="White" />
+      <material name="Purple" />
     </visual>
     <collision>
@@ -97,8 +97,18 @@
           <cylinder length="${base_height}" radius="${base_radius}" />
       </geometry>
+      <surface>
+ <!--###########################-->
+        <friction>
+          <ode>
+            <mu>100</mu>
+            <mu2>100</mu2>
+          </ode>
+        </friction>
+<!--###########################-->
+      </surface>
     </collision>
   </link>
   <gazebo reference="base_link">
-    <material>Gazebo/White</material>
+    <material>Gazebo/Blue</material>
     <turnGravityOff>false</turnGravityOff>
   </gazebo>

Commit message: kinematics detected and put one block completed

File: catkin_yuhaow7/src/drivers/diff_wheeled_robot_gazebo/urdf/diff_wheeled_robot.xacro (robot description, xacro)
@@ -41,5 +41,5 @@
   <xacro:property name="base_z_origin_to_wheel_origin" value="0.0" />
   <!-- Hokuyo Laser scanner -->
-  <xacro:property name="hokuyo_size" value="0.05" />
+  <xacro:property name="hokuyo_size" value="0.01" />
   <!-- Macro for calculating inertia of cylinder -->
   <xacro:macro name="cylinder_inertia" params="m r h">

Commit message: second arm

File: catkin_yuhaow7/src/drivers/diff_wheeled_robot_gazebo/urdf/diff_wheeled_robot.xacro (robot description, xacro)
@@ -120,5 +120,5 @@
 	<sphere radius="${caster_f_radius}" />
       </geometry>
-      <material name="Black" />
+      <material name="Purple" />
     </visual>
       <collision>
@@ -142,4 +142,5 @@
     </joint>
   <gazebo reference="caster_front_link">
+    <material>Gazebo/Blue</material>
     <turnGravityOff>false</turnGravityOff>
   </gazebo>
@@ -151,5 +152,5 @@
 	<sphere radius="${caster_b_radius}" />
       </geometry>
-      <material name="Black" />
+      <material name="Purple" />
     </visual>
       <collision>
@@ -173,4 +174,5 @@
     </joint>
   <gazebo reference="caster_back_link">
+    <material>Gazebo/Blue</material>
     <turnGravityOff>false</turnGravityOff>
   </gazebo>
